Commit message: update still object

File: rrbot_description/urdf/rrbot.xacro (robot description, xacro)
@@ -23,5 +23,5 @@
   <link name="link1">
     <visual>
-      <origin xyz="0 0 ${height1/2}" rpy="0 0 0"/>
+      <origin xyz="0 0 0" rpy="0 0 0"/>
       <geometry>
 	<box size="${width} ${width} ${height1}"/>
@@ -30,5 +30,5 @@
     </visual>
     <inertial>
-      <origin xyz="0 0 ${height1/2}" rpy="0 0 0"/>
+      <origin xyz="0 0 0" rpy="0 0 0"/>
       <mass value="${mass}"/>
       <inertia
@@ -40,5 +40,5 @@
   <joint name="camera_joint" type="fixed">
     <axis xyz="0 1 0" />
-    <origin xyz="${camera_link} 0 ${height3 - axel_offset*2}" rpy="0 0 0"/>
+    <origin xyz="0 0 0" rpy="0 0 0"/>
     <parent link="link1"/>
     <child link="camera_link"/>
